Commit message: pybullet gripper can now pick objects but placing is doing weird stuff

File: urdf/ur5/ur5_w_simple_gripper.urdf (robot description, URDF)
Before this commit: robot assembled_robot, 14 links, 13 joints
Links:
- link simple_gripper_base: mass None -> 1.0
- link simple_gripper_left_finger: mass None -> 0.5
- link simple_gripper_right_finger: mass None -> 0.5

Commit message: More work towards simple gripper working

File: urdf/ur5/ur5_w_simple_gripper.urdf (robot description, URDF)
Before this commit: robot assembled_robot, 14 links, 13 joints
Links:
- added link simple_gripper_tip
- link simple_gripper_left_finger: mass 0.5 -> 1.5
- link simple_gripper_right_finger: mass 0.5 -> 1.5
Joints:
- added joint simple_gripper_tip_joint: type fixed, parent simple_gripper_base, child simple_gripper_tip, origin xyz=0.0 0.0 0.040 rpy=0 0 0

Commit message: increase collision box size

File: urdf/ur5/ur5_w_simple_gripper.urdf (robot description, URDF)
Before this commit: robot assembled_robot, 15 links, 14 joints
Links:
- link simple_gripper_left_finger: geometry collision box size=0.005 0.025 0.06; visual box size=0.005 0.025 0.06
- link simple_gripper_right_finger: geometry collision box size=0.005 0.025 0.06; visual box size=0.005 0.025 0.06

Commit message: add inertial data to dummy link to suppress bullet warning

File: urdf/ur5/ur5_w_simple_gripper.urdf (robot description, URDF)
Before this commit: robot assembled_robot, 15 links, 14 joints
Links:
- link simple_arm_base: mass None -> 0
- link simple_arm_ee_link: mass None -> 0
- link simple_arm_tool0: mass None -> 0
- link simple_gripper_tip: mass None -> 0
