Commit message: integrate ur5_robotiq with robot base class, improve robotiq gripper

File: urdf/ur5/ur5.urdf (robot description, URDF)
Before this commit: robot ur5, 11 links, 10 joints
Links:
- removed link base
- removed link base_link
- removed link ee_link
- removed link forearm_link
- removed link shoulder_link
- removed link tool0
- removed link upper_arm_link
- removed link wrist_1_link
- removed link wrist_2_link
- removed link wrist_3_link
- added link simple_arm_base
- added link simple_arm_base_link, mass 4.0; collision mesh filename=ur5_meshes/base.stl; visual mesh filename=ur5_meshes/base.dae
- added link simple_arm_ee_link; collision box size=0.01 0.01 0.01
- added link simple_arm_forearm_link, mass 2.275; collision mesh filename=ur5_meshes/forearm.stl; visual mesh filename=ur5_meshes/forearm.dae
- added link simple_arm_shoulder_link, mass 3.7; collision mesh filename=ur5_meshes/shoulder.stl; visual mesh filename=ur5_meshes/shoulder.dae
- added link simple_arm_tool0
- added link simple_arm_upper_arm_link, mass 8.393; collision mesh filename=ur5_meshes/upperarm.stl; visual mesh filename=ur5_meshes/upperarm.dae
- added link simple_arm_wrist_1_link, mass 1.219; collision mesh filename=ur5_meshes/wrist1.stl; visual mesh filename=ur5_meshes/wrist1.dae
- added link simple_arm_wrist_2_link, mass 1.219; collision mesh filename=ur5_meshes/wrist2.stl; visual mesh filename=ur5_meshes/wrist2.dae
- added link simple_arm_wrist_3_link, mass 0.1879; collision mesh filename=ur5_meshes/wrist3.stl; visual mesh filename=ur5_meshes/wrist3.dae
Joints:
- removed joint base_link-base_fixed_joint
- removed joint ee_fixed_joint
- removed joint elbow_joint
- removed joint shoulder_lift_joint
- removed joint shoulder_pan_joint
- removed joint wrist_1_joint
- removed joint wrist_2_joint
- removed joint wrist_3_joint
- removed joint wrist_3_link-tool0_fixed_joint
- added joint simple_arm_base_link-base_fixed_joint: type fixed, parent simple_arm_base_link, child simple_arm_base, origin xyz=0 0 0 rpy=0 0 -3.14159265359
- added joint simple_arm_ee_fixed_joint: type fixed, parent simple_arm_wrist_3_link, child simple_arm_ee_link, origin xyz=0.0 0.0823 0.0 rpy=0.0 0.0 1.57079632679
- added joint simple_arm_elbow_joint: type revolute, parent simple_arm_upper_arm_link, child simple_arm_forearm_link, origin xyz=0.0 -0.1197 0.425 rpy=0.0 0.0 0.0, axis 0 1 0, limit lower=-3.14159265359 upper=3.14159265359 effort=150.0 velocity=3.15
- added joint simple_arm_shoulder_lift_joint: type revolute, parent simple_arm_shoulder_link, child simple_arm_upper_arm_link, origin xyz=0.0 0.13585 0.0 rpy=0.0 1.57079632679 0.0, axis 0 1 0, limit lower=-6.28318530718 upper=6.28318530718 effort=150.0 velocity=3.15
- added joint simple_arm_shoulder_pan_joint: type revolute, parent simple_arm_base_link, child simple_arm_shoulder_link, origin xyz=0.0 0.0 0.089159 rpy=0.0 0.0 0.0, axis 0 0 1, limit lower=-6.28318530718 upper=6.28318530718 effort=150.0 velocity=3.15
- added joint simple_arm_wrist_1_joint: type revolute, parent simple_arm_forearm_link, child simple_arm_wrist_1_link, origin xyz=0.0 0.0 0.39225 rpy=0.0 1.57079632679 0.0, axis 0 1 0, limit lower=-6.28318530718 upper=6.28318530718 effort=28.0 velocity=3.2
- added joint simple_arm_wrist_2_joint: type revolute, parent simple_arm_wrist_1_link, child simple_arm_wrist_2_link, origin xyz=0.0 0.093 0.0 rpy=0.0 0.0 0.0, axis 0 0 1, limit lower=-6.28318530718 upper=6.28318530718 effort=28.0 velocity=3.2
- added joint simple_arm_wrist_3_joint: type revolute, parent simple_arm_wrist_2_link, child simple_arm_wrist_3_link, origin xyz=0.0 0.0 0.09465 rpy=0.0 0.0 0.0, axis 0 1 0, limit lower=-6.28318530718 upper=6.28318530718 effort=28.0 velocity=3.2
- added joint simple_arm_wrist_3_link-tool0_fixed_joint: type fixed, parent simple_arm_wrist_3_link, child simple_arm_tool0, origin xyz=0 0.0823 0 rpy=-1.57079632679 0 0
- joint world_joint: child base_link -> simple_arm_base_link

File: urdf/ur5/ur5_w_robotiq_85_gripper.urdf (robot description, URDF)
Before this commit: robot assembled_robot, 21 links, 20 joints
Links:
- link robotiq_85_left_finger_link: mass 0.027309 -> 0.27309
- link robotiq_85_left_finger_tip_link: mass 0.019555 -> 0.19555
- link robotiq_85_left_inner_knuckle_link: mass 0.029951 -> 0.29951
- link robotiq_85_left_knuckle_link: mass 0.018491 -> 0.18491
- link robotiq_85_right_finger_link: mass 0.027309 -> 0.27309
- link robotiq_85_right_finger_tip_link: mass 0.019555 -> 0.19555
- link robotiq_85_right_inner_knuckle_link: mass 0.029951 -> 0.29951
- link robotiq_85_right_knuckle_link: mass 0.018491 -> 0.18491
- link simple_arm_base: mass None -> 0
- link simple_arm_ee_link: mass None -> 0
- link simple_arm_tool0: mass None -> 0
Joints:
- joint dummy_center_fixed_joint: origin xyz=0.14 0 0 -> xyz=0.14 0 0 rpy=0.0 1.5707 0.0
- joint robotiq_85_left_finger_tip_joint: limit lower=-3.14 upper=3.14 effort=0.3 velocity=3.14 -> lower=-3.14 upper=3.14 effort=2 velocity=3.14
- joint robotiq_85_left_inner_knuckle_joint: limit lower=-3.14 upper=3.14 effort=0.3 velocity=3.14 -> lower=-3.14 upper=3.14 effort=2 velocity=3.14
- joint robotiq_85_right_finger_tip_joint: limit lower=-3.14 upper=3.14 effort=0.3 velocity=3.14 -> lower=-3.14 upper=3.14 effort=2 velocity=3.14
- joint robotiq_85_right_inner_knuckle_joint: limit lower=-3.14 upper=3.14 effort=0.3 velocity=3.14 -> lower=-3.14 upper=3.14 effort=2 velocity=3.14
