Commit message: toward adding robotiq85 gripper

File: urdf/ur5/ur5_w_robotiq_85_gripper.urdf (robot description, URDF)
Before this commit: robot assembled_robot, 22 links, 21 joints
Links:
- removed link simple_gripper_base
- removed link simple_gripper_left_coupler
- removed link simple_gripper_left_driver
- removed link simple_gripper_left_follower
- removed link simple_gripper_left_pad
- removed link simple_gripper_left_spring_link
- removed link simple_gripper_right_coupler
- removed link simple_gripper_right_driver
- removed link simple_gripper_right_follower
- removed link simple_gripper_right_pad
- removed link simple_gripper_right_spring_link
- added link robotiq_85_base_link, mass 0.636951; collision mesh filename=../meshes/collision/robotiq_85_base_link.stl; visual mesh filename=../meshes/visual/robotiq_85_base_link.dae
- added link robotiq_85_left_finger_link, mass 0.027309; collision mesh filename=../meshes/collision/robotiq_85_finger_link.stl; visual mesh filename=../meshes/visual/robotiq_85_finger_link.dae
- added link robotiq_85_left_finger_tip_link, mass 0.019555; collision mesh filename=../meshes/collision/robotiq_85_finger_tip_link.stl; visual mesh filename=../meshes/visual/robotiq_85_finger_tip_link.dae
- added link robotiq_85_left_inner_knuckle_link, mass 0.029951; collision mesh filename=../meshes/collision/robotiq_85_inner_knuckle_link.stl; visual mesh filename=../meshes/visual/robotiq_85_inner_knuckle_link.dae
- added link robotiq_85_left_knuckle_link, mass 0.018491; collision mesh filename=../meshes/collision/robotiq_85_knuckle_link.stl; visual mesh filename=../meshes/visual/robotiq_85_knuckle_link.dae
- added link robotiq_85_right_finger_link, mass 0.027309; collision mesh filename=../meshes/collision/robotiq_85_finger_link.stl; visual mesh filename=../meshes/visual/robotiq_85_finger_link.dae
- added link robotiq_85_right_finger_tip_link, mass 0.019555; collision mesh filename=../meshes/collision/robotiq_85_finger_tip_link.stl; visual mesh filename=../meshes/visual/robotiq_85_finger_tip_link.dae
- added link robotiq_85_right_inner_knuckle_link, mass 0.029951; collision mesh filename=../meshes/collision/robotiq_85_inner_knuckle_link.stl; visual mesh filename=../meshes/visual/robotiq_85_inner_knuckle_link.dae
- added link robotiq_85_right_knuckle_link, mass 0.018491; collision mesh filename=../meshes/collision/robotiq_85_knuckle_link.stl; visual mesh filename=../meshes/visual/robotiq_85_knuckle_link.dae
Joints:
- removed joint simple_gripper_left_coupler_joint
- removed joint simple_gripper_left_driver_joint
- removed joint simple_gripper_left_follower_joint
- removed joint simple_gripper_left_pad_joint
- removed joint simple_gripper_left_spring_link_joint
- removed joint simple_gripper_right_coupler_joint
- removed joint simple_gripper_right_driver_joint
- removed joint simple_gripper_right_follower_joint
- removed joint simple_gripper_right_pad_joint
- removed joint simple_gripper_right_spring_link_joint
- added joint robotiq_85_left_finger_joint: type fixed, parent robotiq_85_left_knuckle_link, child robotiq_85_left_finger_link, origin xyz=-0.00408552455 -0.03148604435 0.0 rpy=0 0 0
- added joint robotiq_85_left_finger_tip_joint: type revolute, parent robotiq_85_left_inner_knuckle_link, child robotiq_85_left_finger_tip_link, origin xyz=0.04303959807 -0.03759940821 0.0 rpy=0.0 0.0 0.0, axis 0 0 1, limit lower=-3.14 upper=3.14 effort=0.1 velocity=3.14, mimic joint=robotiq_85_left_knuckle_joint multiplier=-1
- added joint robotiq_85_left_inner_knuckle_joint: type revolute, parent robotiq_85_base_link, child robotiq_85_left_inner_knuckle_link, origin xyz=0.06142 0.0127 0 rpy=3.14 0.0 0.0, axis 0 0 1, limit lower=-3.14 upper=3.14 effort=0.1 velocity=3.14, mimic joint=robotiq_85_left_knuckle_joint offset=0
- added joint robotiq_85_left_knuckle_joint: type revolute, parent robotiq_85_base_link, child robotiq_85_left_knuckle_link, origin xyz=0.05490451627 0.03060114443 0.0 rpy=3.14 0.0 0.0, axis 0 0 1, limit lower=0.0 upper=0.80285 effort=1000 velocity=3.14
- added joint robotiq_85_right_finger_joint: type fixed, parent robotiq_85_right_knuckle_link, child robotiq_85_right_finger_link, origin xyz=-0.00408552455 -0.03148604435 0.0 rpy=0 0 0
- added joint robotiq_85_right_finger_tip_joint: type revolute, parent robotiq_85_right_inner_knuckle_link, child robotiq_85_right_finger_tip_link, origin xyz=0.04303959807 -0.03759940821  0.0 rpy=0.0 0.0 0.0, axis 0 0 1, limit lower=-3.14 upper=3.14 effort=0.1 velocity=3.14, mimic joint=robotiq_85_left_knuckle_joint multiplier=-1
- added joint robotiq_85_right_inner_knuckle_joint: type revolute, parent robotiq_85_base_link, child robotiq_85_right_inner_knuckle_link, origin xyz=0.06142 -0.0127 0 rpy=0 0 0, axis 0 0 1, limit lower=-3.14 upper=3.14 effort=0.1 velocity=3.14, mimic joint=robotiq_85_left_knuckle_joint offset=0
- added joint robotiq_85_right_knuckle_joint: type revolute, parent robotiq_85_base_link, child robotiq_85_right_knuckle_link, origin xyz=0.05490451627 -0.03060114443 0.0 rpy=0.0 0.0 0.0, axis 0 0 1, limit lower=-3.14 upper=3.14 effort=1000 velocity=3.14, mimic joint=robotiq_85_left_knuckle_joint
- joint simple_arm_tool0_simple_gripper_base_joint: child simple_gripper_base -> robotiq_85_base_link; origin xyz=0 0 0 rpy=0 0 1.5708 -> xyz=0 0 0 rpy=0 -1.5708 0

Commit message: grasping not stable

File: urdf/ur5/ur5_w_robotiq_85_gripper.urdf (robot description, URDF)
Before this commit: robot assembled_robot, 20 links, 19 joints
Links:
- added link dummy_center_indicator_link, mass 0.0
Joints:
- added joint dummy_center_fixed_joint: type fixed, parent robotiq_85_base_link, child dummy_center_indicator_link, origin xyz=0.14 0 0
- joint robotiq_85_left_finger_tip_joint: limit lower=-3.14 upper=3.14 effort=0.1 velocity=3.14 -> lower=-3.14 upper=3.14 effort=0.3 velocity=3.14
- joint robotiq_85_left_inner_knuckle_joint: limit lower=-3.14 upper=3.14 effort=0.1 velocity=3.14 -> lower=-3.14 upper=3.14 effort=0.3 velocity=3.14
- joint robotiq_85_right_finger_tip_joint: limit lower=-3.14 upper=3.14 effort=0.1 velocity=3.14 -> lower=-3.14 upper=3.14 effort=0.3 velocity=3.14
- joint robotiq_85_right_inner_knuckle_joint: limit lower=-3.14 upper=3.14 effort=0.1 velocity=3.14 -> lower=-3.14 upper=3.14 effort=0.3 velocity=3.14

Commit message: play with parameters

File: urdf/ur5/ur5_w_robotiq_85_gripper.urdf (robot description, URDF)
Before this commit: robot assembled_robot, 21 links, 20 joints
Joints:
- joint robotiq_85_left_finger_tip_joint: limit lower=-3.14 upper=3.14 effort=2 velocity=3.14 -> lower=-3.14 upper=3.14 effort=10 velocity=3.14
- joint robotiq_85_left_inner_knuckle_joint: limit lower=-3.14 upper=3.14 effort=2 velocity=3.14 -> lower=-3.14 upper=3.14 effort=20 velocity=3.14
- joint robotiq_85_right_finger_tip_joint: limit lower=-3.14 upper=3.14 effort=2 velocity=3.14 -> lower=-3.14 upper=3.14 effort=10 velocity=3.14
- joint robotiq_85_right_inner_knuckle_joint: limit lower=-3.14 upper=3.14 effort=2 velocity=3.14 -> lower=-3.14 upper=3.14 effort=20 velocity=3.14
