Commit message: use box to replace finger tip

File: simulators/urdf/ur5/ur5_robotiq_85_gripper.urdf (robot description, URDF)
Before this commit: robot assembled_robot, 21 links, 20 joints
Links:
- link robotiq_85_left_finger_tip_link: mass 0.19555 -> 1; geometry collision box size=0.05 0.005 0.025; visual box size=0.05 0.005 0.025
- link robotiq_85_right_finger_tip_link: mass 0.19555 -> 1; geometry collision box size=0.05 0.005 0.025; visual box size=0.05 0.005 0.025
Joints:
- joint dummy_center_fixed_joint: origin xyz=0.14 0 0 rpy=0.0 1.5707 0.0 -> xyz=0 0 0.14 rpy=0.0 0.0 1.5707; parent robotiq_85_base_link -> simple_arm_tool0
- joint robotiq_85_left_finger_tip_joint: limit lower=-3.14 upper=3.14 effort=10 velocity=3.14 -> lower=-3.14 upper=3.14 effort=60 velocity=0.02; origin xyz=0.04303959807 -0.03759940821 0.0 rpy=0.0 0.0 0.0 -> xyz=0.064 -0.03759940821  0.0 rpy=0.0 0.0 0.0
- joint robotiq_85_left_inner_knuckle_joint: limit lower=-3.14 upper=3.14 effort=20 velocity=3.14 -> lower=-3.14 upper=3.14 effort=60 velocity=3.14
- joint robotiq_85_right_finger_tip_joint: limit lower=-3.14 upper=3.14 effort=10 velocity=3.14 -> lower=-3.14 upper=3.14 effort=60 velocity=0.02; origin xyz=0.04303959807 -0.03759940821  0.0 rpy=0.0 0.0 0.0 -> xyz=0.064 -0.03759940821  0.0 rpy=0.0 0.0 0.0
- joint robotiq_85_right_inner_knuckle_joint: limit lower=-3.14 upper=3.14 effort=20 velocity=3.14 -> lower=-3.14 upper=3.14 effort=60 velocity=3.14
