Commit message: minor changes

File: simulators/urdf/ur5/ur5_robotiq_85_gripper_fake.urdf (robot description, URDF)
Before this commit: robot assembled_robot, 25 links, 24 joints
Links:
- link simple_gripper_base: geometry collision box size=0.005 0.0025 0.005

Commit message: restore the changes in place_offset; decrease finger tip width to 0.02

File: simulators/urdf/ur5/ur5_robotiq_85_gripper_fake.urdf (robot description, URDF)
Before this commit: robot assembled_robot, 25 links, 24 joints
Links:
- link simple_gripper_left_finger: geometry collision box size=0.005 0.02 0.06; visual box size=0.005 0.02 0.06
- link simple_gripper_right_finger: geometry collision box size=0.005 0.02 0.06; visual box size=0.005 0.02 0.06
