Commit message: change the z scale of random objs; add check_random_obj_valid flag

File: simulators/urdf/object/random_urdfs/000/000.urdf (robot description, URDF)
Before this commit: robot blob000, 1 links, 0 joints
Links:
- link random_obj_000: geometry collision mesh filename=000.obj scale=0.015 0.015 0.01; visual mesh filename=000.obj scale=0.015 0.015 0.01

File: simulators/urdf/object/random_urdfs/000/000_2.urdf (robot description, URDF)
Before this commit: robot blob000, 1 links, 0 joints
Links:
- link random_obj_000: geometry collision mesh filename=000.obj scale=0.015 0.015 0.02; visual mesh filename=000.obj scale=0.015 0.015 0.02

File: simulators/urdf/object/random_urdfs/001/001.urdf (robot description, URDF)
Before this commit: robot blob001, 1 links, 0 joints
Links:
- link random_obj_001: geometry collision mesh filename=001.obj scale=0.015 0.015 0.01; visual mesh filename=001.obj scale=0.015 0.015 0.01

File: simulators/urdf/object/random_urdfs/001/001_2.urdf (robot description, URDF)
Before this commit: robot blob001, 1 links, 0 joints
Links:
- link random_obj_001: geometry collision mesh filename=001.obj scale=0.015 0.015 0.02; visual mesh filename=001.obj scale=0.015 0.015 0.02

File: simulators/urdf/object/random_urdfs/002/002.urdf (robot description, URDF)
Before this commit: robot blob002, 1 links, 0 joints
Links:
- link random_obj_002: geometry collision mesh filename=002.obj scale=0.015 0.015 0.01; visual mesh filename=002.obj scale=0.015 0.015 0.01

File: simulators/urdf/object/random_urdfs/002/002_2.urdf (robot description, URDF)
Before this commit: robot blob002, 1 links, 0 joints
Links:
- link random_obj_002: geometry collision mesh filename=002.obj scale=0.015 0.015 0.02; visual mesh filename=002.obj scale=0.015 0.015 0.02

File: simulators/urdf/object/random_urdfs/003/003.urdf (robot description, URDF)
Before this commit: robot blob003, 1 links, 0 joints
Links:
- link random_obj_003: geometry collision mesh filename=003.obj scale=0.015 0.015 0.01; visual mesh filename=003.obj scale=0.015 0.015 0.01

File: simulators/urdf/object/random_urdfs/003/003_2.urdf (robot description, URDF)
Before this commit: robot blob003, 1 links, 0 joints
Links:
- link random_obj_003: geometry collision mesh filename=003.obj scale=0.015 0.015 0.02; visual mesh filename=003.obj scale=0.015 0.015 0.02

File: simulators/urdf/object/random_urdfs/004/004.urdf (robot description, URDF)
Before this commit: robot blob004, 1 links, 0 joints
Links:
- link random_obj_004: geometry collision mesh filename=004.obj scale=0.015 0.015 0.01; visual mesh filename=004.obj scale=0.015 0.015 0.01

File: simulators/urdf/object/random_urdfs/004/004_2.urdf (robot description, URDF)
Before this commit: robot blob004, 1 links, 0 joints
Links:
- link random_obj_004: geometry collision mesh filename=004.obj scale=0.015 0.015 0.02; visual mesh filename=004.obj scale=0.015 0.015 0.02

File: simulators/urdf/object/random_urdfs/005/005.urdf (robot description, URDF)
Before this commit: robot blob005, 1 links, 0 joints
Links:
- link random_obj_005: geometry collision mesh filename=005.obj scale=0.015 0.015 0.01; visual mesh filename=005.obj scale=0.015 0.015 0.01

File: simulators/urdf/object/random_urdfs/005/005_2.urdf (robot description, URDF)
Before this commit: robot blob005, 1 links, 0 joints
Links:
- link random_obj_005: geometry collision mesh filename=005.obj scale=0.015 0.015 0.02; visual mesh filename=005.obj scale=0.015 0.015 0.02

File: simulators/urdf/object/random_urdfs/006/006.urdf (robot description, URDF)
Before this commit: robot blob006, 1 links, 0 joints
Links:
- link random_obj_006: geometry collision mesh filename=006.obj scale=0.015 0.015 0.01; visual mesh filename=006.obj scale=0.015 0.015 0.01

File: simulators/urdf/object/random_urdfs/006/006_2.urdf (robot description, URDF)
Before this commit: robot blob006, 1 links, 0 joints
Links:
- link random_obj_006: geometry collision mesh filename=006.obj scale=0.015 0.015 0.02; visual mesh filename=006.obj scale=0.015 0.015 0.02

File: simulators/urdf/object/random_urdfs/007/007.urdf (robot description, URDF)
Before this commit: robot blob007, 1 links, 0 joints
Links:
- link random_obj_007: geometry collision mesh filename=007.obj scale=0.015 0.015 0.01; visual mesh filename=007.obj scale=0.015 0.015 0.01

File: simulators/urdf/object/random_urdfs/007/007_2.urdf (robot description, URDF)
Before this commit: robot blob007, 1 links, 0 joints
Links:
- link random_obj_007: geometry collision mesh filename=007.obj scale=0.015 0.015 0.02; visual mesh filename=007.obj scale=0.015 0.015 0.02

File: simulators/urdf/object/random_urdfs/008/008.urdf (robot description, URDF)
Before this commit: robot blob008, 1 links, 0 joints
Links:
- link random_obj_008: geometry collision mesh filename=008.obj scale=0.015 0.015 0.01; visual mesh filename=008.obj scale=0.015 0.015 0.01

File: simulators/urdf/object/random_urdfs/008/008_2.urdf (robot description, URDF)
Before this commit: robot blob008, 1 links, 0 joints
Links:
- link random_obj_008: geometry collision mesh filename=008.obj scale=0.015 0.015 0.02; visual mesh filename=008.obj scale=0.015 0.015 0.02

File: simulators/urdf/object/random_urdfs/009/009.urdf (robot description, URDF)
Before this commit: robot blob009, 1 links, 0 joints
Links:
- link random_obj_009: geometry collision mesh filename=009.obj scale=0.015 0.015 0.01; visual mesh filename=009.obj scale=0.015 0.015 0.01

File: simulators/urdf/object/random_urdfs/009/009_2.urdf (robot description, URDF)
Before this commit: robot blob009, 1 links, 0 joints
Links:
- link random_obj_009: geometry collision mesh filename=009.obj scale=0.015 0.015 0.02; visual mesh filename=009.obj scale=0.015 0.015 0.02
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
Commit message: decrease the xy extensions of random objs

File: simulators/urdf/object/random_urdfs/000/000.urdf (robot description, URDF)
Before this commit: robot blob000, 1 links, 0 joints
Links:
- link random_obj_000: geometry collision mesh filename=000.obj scale=0.012 0.012 0.01; visual mesh filename=000.obj scale=0.012 0.012 0.01

File: simulators/urdf/object/random_urdfs/000/000_2.urdf (robot description, URDF)
Before this commit: robot blob000, 1 links, 0 joints
Links:
- link random_obj_000: geometry collision mesh filename=000.obj scale=0.012 0.012 0.02; visual mesh filename=000.obj scale=0.012 0.012 0.02

File: simulators/urdf/object/random_urdfs/001/001.urdf (robot description, URDF)
Before this commit: robot blob001, 1 links, 0 joints
Links:
- link random_obj_001: geometry collision mesh filename=001.obj scale=0.012 0.012 0.01; visual mesh filename=001.obj scale=0.012 0.012 0.01

File: simulators/urdf/object/random_urdfs/001/001_2.urdf (robot description, URDF)
Before this commit: robot blob001, 1 links, 0 joints
Links:
- link random_obj_001: geometry collision mesh filename=001.obj scale=0.012 0.012 0.02; visual mesh filename=001.obj scale=0.012 0.012 0.02

File: simulators/urdf/object/random_urdfs/002/002.urdf (robot description, URDF)
Before this commit: robot blob002, 1 links, 0 joints
Links:
- link random_obj_002: geometry collision mesh filename=002.obj scale=0.012 0.012 0.01; visual mesh filename=002.obj scale=0.012 0.012 0.01

File: simulators/urdf/object/random_urdfs/002/002_2.urdf (robot description, URDF)
Before this commit: robot blob002, 1 links, 0 joints
Links:
- link random_obj_002: geometry collision mesh filename=002.obj scale=0.012 0.012 0.02; visual mesh filename=002.obj scale=0.012 0.012 0.02

File: simulators/urdf/object/random_urdfs/003/003.urdf (robot description, URDF)
Before this commit: robot blob003, 1 links, 0 joints
Links:
- link random_obj_003: geometry collision mesh filename=003.obj scale=0.012 0.012 0.01; visual mesh filename=003.obj scale=0.012 0.012 0.01

File: simulators/urdf/object/random_urdfs/003/003_2.urdf (robot description, URDF)
Before this commit: robot blob003, 1 links, 0 joints
Links:
- link random_obj_003: geometry collision mesh filename=003.obj scale=0.012 0.012 0.02; visual mesh filename=003.obj scale=0.012 0.012 0.02

File: simulators/urdf/object/random_urdfs/004/004.urdf (robot description, URDF)
Before this commit: robot blob004, 1 links, 0 joints
Links:
- link random_obj_004: geometry collision mesh filename=004.obj scale=0.012 0.012 0.01; visual mesh filename=004.obj scale=0.012 0.012 0.01

File: simulators/urdf/object/random_urdfs/004/004_2.urdf (robot description, URDF)
Before this commit: robot blob004, 1 links, 0 joints
Links:
- link random_obj_004: geometry collision mesh filename=004.obj scale=0.012 0.012 0.02; visual mesh filename=004.obj scale=0.012 0.012 0.02

File: simulators/urdf/object/random_urdfs/005/005.urdf (robot description, URDF)
Before this commit: robot blob005, 1 links, 0 joints
Links:
- link random_obj_005: geometry collision mesh filename=005.obj scale=0.012 0.012 0.01; visual mesh filename=005.obj scale=0.012 0.012 0.01

File: simulators/urdf/object/random_urdfs/005/005_2.urdf (robot description, URDF)
Before this commit: robot blob005, 1 links, 0 joints
Links:
- link random_obj_005: geometry collision mesh filename=005.obj scale=0.012 0.012 0.02; visual mesh filename=005.obj scale=0.012 0.012 0.02

File: simulators/urdf/object/random_urdfs/006/006.urdf (robot description, URDF)
Before this commit: robot blob006, 1 links, 0 joints
Links:
- link random_obj_006: geometry collision mesh filename=006.obj scale=0.012 0.012 0.01; visual mesh filename=006.obj scale=0.012 0.012 0.01

File: simulators/urdf/object/random_urdfs/006/006_2.urdf (robot description, URDF)
Before this commit: robot blob006, 1 links, 0 joints
Links:
- link random_obj_006: geometry collision mesh filename=006.obj scale=0.012 0.012 0.02; visual mesh filename=006.obj scale=0.012 0.012 0.02

File: simulators/urdf/object/random_urdfs/007/007.urdf (robot description, URDF)
Before this commit: robot blob007, 1 links, 0 joints
Links:
- link random_obj_007: geometry collision mesh filename=007.obj scale=0.012 0.012 0.01; visual mesh filename=007.obj scale=0.012 0.012 0.01

File: simulators/urdf/object/random_urdfs/007/007_2.urdf (robot description, URDF)
Before this commit: robot blob007, 1 links, 0 joints
Links:
- link random_obj_007: geometry collision mesh filename=007.obj scale=0.012 0.012 0.02; visual mesh filename=007.obj scale=0.012 0.012 0.02

File: simulators/urdf/object/random_urdfs/008/008.urdf (robot description, URDF)
Before this commit: robot blob008, 1 links, 0 joints
Links:
- link random_obj_008: geometry collision mesh filename=008.obj scale=0.012 0.012 0.01; visual mesh filename=008.obj scale=0.012 0.012 0.01

File: simulators/urdf/object/random_urdfs/008/008_2.urdf (robot description, URDF)
Before this commit: robot blob008, 1 links, 0 joints
Links:
- link random_obj_008: geometry collision mesh filename=008.obj scale=0.012 0.012 0.02; visual mesh filename=008.obj scale=0.012 0.012 0.02

File: simulators/urdf/object/random_urdfs/009/009.urdf (robot description, URDF)
Before this commit: robot blob009, 1 links, 0 joints
Links:
- link random_obj_009: geometry collision mesh filename=009.obj scale=0.012 0.012 0.01; visual mesh filename=009.obj scale=0.012 0.012 0.01

File: simulators/urdf/object/random_urdfs/009/009_2.urdf (robot description, URDF)
Before this commit: robot blob009, 1 links, 0 joints
Links:
- link random_obj_009: geometry collision mesh filename=009.obj scale=0.012 0.012 0.02; visual mesh filename=009.obj scale=0.012 0.012 0.02
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