Commit message: remove 'side_grasp' and 'side_place' in planners, change the object urdf s.t. they can be picked up at 0 orientation

File: simulators/urdf/object/brick_small.urdf (robot description, URDF)
Before this commit: robot cube.urdf, 1 links, 0 joints
Links:
- link baseLink: geometry collision box size=.05 .15 .05; visual mesh filename=cube.obj scale=.05 .15 .05
