Commit message: Changes urdf block to be more realistic

File: simulators/urdf/object/cube.urdf (robot description, URDF)
Before this commit: robot cube.urdf, 1 links, 0 joints
Links:
- link baseLink: mass 0.1 -> 0.05; geometry collision box size=0.05 0.05 0.05; visual mesh filename=cube.obj scale=0.05 0.05 0.05

Commit message: New cube urdf to help edge cases

File: simulators/urdf/object/cube.urdf (robot description, URDF)
Before this commit: robot cube, 1 links, 0 joints
Links:
- link baseLink: mass 0.05 -> 0.1

Commit message: More attempts to stabalize the simulation

File: simulators/urdf/object/cube.urdf (robot description, URDF)
Before this commit: robot cube, 1 links, 0 joints
Links:
- link baseLink: mass 0.1 -> 0.10

Commit message: Lots of small changes to get more stable simulations, seems like this was mostly due to how the kuka gripper was opening/closing. Current fix is to sse the stabalize the block while the gripper opens and then allow dynamics to start effecting it again. Will need a better solution going forward however. Additional changes to stabalize the env may or may not be needed but it seems good to have them in so they are staying for the moment.

File: simulators/urdf/object/cube.urdf (robot description, URDF)
Before this commit: robot cube, 1 links, 0 joints
Links:
- link baseLink: mass 0.10 -> 0.1; geometry collision box size=0.05 0.05 0.05; visual box size=0.05 0.05 0.05
