Commit message: Made a couple of small changes to the pybullet object classes and the corresponding urdfs

File: simulators/urdf/object/cylinder.urdf (robot description, URDF)
Before this commit: robot cylinder.urdf, 1 links, 0 joints
Links:
- link baseLink: geometry collision mesh filename=cylinder.obj scale=0.5 0.5 0.5; visual mesh filename=cylinder.obj scale=0.5 0.5 0.5
