Commit message: match the ori of upper cubes in h4 deconstruct to reduce the chance of collision. Increase the size of ramp for 128 exps

File: simulators/urdf/object/tilt.urdf (robot description, URDF)
Before this commit: robot tilt.urdf, 1 links, 0 joints
Links:
- link baseLink: geometry collision box size=0.6 0.3 .01; visual box size=0.6 0.3 .01
