Commit message: remove the grasp helper cube's visual shape in teapots and lids

File: simulators/urdf/teapot/1/base.urdf (robot description, URDF)
Before this commit: robot partnet_3e47ee246f89d6cdeb5a654451d3cffd-0, 1 links, 0 joints
Links:
- link link_1: geometry collision box size=.3 .3 .3; collision mesh filename=textured_objs/original-1.obj

File: simulators/urdf/teapot/1/lid.urdf (robot description, URDF)
Before this commit: robot partnet_3e47ee246f89d6cdeb5a654451d3cffd-0, 1 links, 0 joints
Links:
- link link_1: geometry collision box size=.3 .3 .2; collision mesh filename=textured_objs/original-3.obj

File: simulators/urdf/teapot/2/base.urdf (robot description, URDF)
Before this commit: robot partnet_464e9b98-d955-4597-b746-4e8b73eab34b, 1 links, 0 joints
Links:
- link link_1: geometry collision box size=.3 .3 .3; collision mesh filename=textured_objs/original-1.obj

File: simulators/urdf/teapot/2/lid.urdf (robot description, URDF)
Before this commit: robot partnet_464e9b98-d955-4597-b746-4e8b73eab34b, 1 links, 0 joints
Links:
- link link_0: geometry collision box size=.3 .3 .2; collision mesh filename=textured_objs/original-5.obj

File: simulators/urdf/teapot/3/base.urdf (robot description, URDF)
Before this commit: robot partnet_50771bde64eff3ac27a11dcb35000f7a-0, 1 links, 0 joints
Links:
- link link_1: geometry collision box size=.3 .3 .3; collision mesh filename=textured_objs/original-2.obj

File: simulators/urdf/teapot/3/lid.urdf (robot description, URDF)
Before this commit: robot partnet_50771bde64eff3ac27a11dcb35000f7a-0, 1 links, 0 joints
Links:
- link link_0: geometry collision box size=.3 .3 .2; collision mesh filename=textured_objs/original-1.obj

File: simulators/urdf/teapot/4/base.urdf (robot description, URDF)
Before this commit: robot partnet_c7a70db33a8c900dab5b523beb03efcd, 1 links, 0 joints
Links:
- link link_1: geometry collision box size=.3 .3 .3; collision mesh filename=textured_objs/original-3.obj

File: simulators/urdf/teapot/4/lid.urdf (robot description, URDF)
Before this commit: robot partnet_c7a70db33a8c900dab5b523beb03efcd, 1 links, 0 joints
Links:
- link link_0: geometry collision box size=.3 .3 .2; collision mesh filename=textured_objs/original-2.obj

File: simulators/urdf/teapot/5/base.urdf (robot description, URDF)
Before this commit: robot partnet_58d1e344ef8364b225e0f641bff885da, 1 links, 0 joints
Links:
- link link_1: geometry collision box size=.3 .3 .3; collision mesh filename=textured_objs/original-1.obj

File: simulators/urdf/teapot/5/lid.urdf (robot description, URDF)
Before this commit: robot partnet_58d1e344ef8364b225e0f641bff885da, 1 links, 0 joints
Links:
- link link_0: geometry collision box size=.3 .3 .2; collision mesh filename=textured_objs/original-2.obj
