Commit message: add drawer_opening env

File: simulators/urdf/drawer.urdf (robot description, URDF)
Before this commit: robot drawer, 16 links, 15 joints
Links:
- link base_link: mass None -> .1
- link drawer: mass None -> .1

Commit message: implement horizontal pull in drawer env, add primative in closeGripper function to adjust force for pick and pull. drawer_opening_env now working

File: simulators/urdf/drawer.urdf (robot description, URDF)
Before this commit: robot drawer, 16 links, 15 joints
Links:
- link handle_grip: geometry collision box size=0.04 0.24 0.04; visual box size=0.04 0.24 0.04
- link handle_left: geometry collision box size=0.06 0.04 0.04; visual box size=0.06 0.04 0.04
- link handle_right: geometry collision box size=0.06 0.04 0.04; visual box size=0.06 0.04 0.04
Joints:
- joint d_2_hl: origin xyz=0.38 -0.085 0 rpy=0 0 0 -> xyz=0.38 -0.1 0 rpy=0 0 0
- joint d_2_hr: origin xyz=0.38 0.085 0 rpy=0 0 0 -> xyz=0.38 0.1 0 rpy=0 0 0

Commit message: working on two drawers

File: simulators/urdf/drawer.urdf (robot description, URDF)
Before this commit: robot drawer, 16 links, 15 joints
Joints:
- joint world_to_base: origin xyz=0 0 0.2 rpy=0 0 3.1415 -> xyz=0 0 0.18 rpy=0 0 3.1415

Commit message: add another teapot model; randomize drawer handle by separating it from the drawer model

File: simulators/urdf/drawer.urdf (robot description, URDF)
Before this commit: robot drawer, 16 links, 15 joints
Links:
- removed link handle_grip
- removed link handle_left
- removed link handle_right
Joints:
- removed joint d_2_hg
- removed joint d_2_hl
- removed joint d_2_hr

Commit message: Improve the speed of point cloud projection to depth image; get the drawer env working with random drawer theta.

File: simulators/urdf/drawer.urdf (robot description, URDF)
Before this commit: robot drawer, 13 links, 12 joints
Links:
- added link drawer_obj_pos, mass 0.05
Joints:
- added joint dbow2dop: type fixed, parent drawer_bottom_wall, child drawer_obj_pos, origin xyz=0.16 0 0.06 rpy=0 0 0

Commit message: increase the horizontal size of the drawer, minor improvement of the drawer teapot planner

File: simulators/urdf/drawer.urdf (robot description, URDF)
Before this commit: robot drawer, 14 links, 13 joints
Links:
- link back_wall: geometry collision box size=0.02 0.76 0.36; visual box size=0.02 0.76 0.36
- link bottom_wall: geometry collision box size=0.71 0.76 0.02; visual box size=0.71 0.76 0.02
- link drawer_back_wall: geometry collision box size=0.02 0.7 0.3; visual box size=0.02 0.7 0.3
- link drawer_bottom_wall: geometry collision box size=0.7 0.7 0.02; visual box size=0.7 0.7 0.02
- link drawer_front_wall: geometry collision box size=0.02 0.7 0.3; visual box size=0.02 0.7 0.3
- link top_wall: geometry collision box size=0.71 0.76 0.02; visual box size=0.71 0.76 0.02
Joints:
- joint b_2_lw: origin xyz=-0.01 -0.32 0 rpy=0 0 0 -> xyz=-0.01 -0.37 0 rpy=0 0 0
- joint b_2_rw: origin xyz=-0.01 0.32 0 rpy=0 0 0 -> xyz=-0.01 0.37 0 rpy=0 0 0
- joint drawer_2_dlw: origin xyz=0 -0.29 0 rpy=0 0 0 -> xyz=0 -0.34 0 rpy=0 0 0
- joint drawer_2_drw: origin xyz=0 0.29 0 rpy=0 0 0 -> xyz=0 0.34 0 rpy=0 0 0
