Commit message: randomize bowl picking point (instead of always pick and place at the same relative point)

File: helping_hands_rl_envs/simulators/urdf/object/bowl/bowl2.urdf (robot description, URDF)
Before this commit: robot bowl.urdf, 2 links, 1 joints
Links:
- link baseLink: geometry collision mesh filename=bowl2.obj scale=0.2 0.2 0.2; visual mesh filename=bowl2.obj scale=0.2 0.2 0.2
Joints:
- joint base2grasp: origin xyz=0.09 0 0 rpy=0 0 0 -> xyz=0.09 0 0.02 rpy=0 0 0
