Commit message: add a cylinder bottom shape in plate1.urdf to reduce the number of contacts

File: helping_hands_rl_envs/simulators/urdf/object/plate/plate1.urdf (robot description, URDF)
Before this commit: robot plate1.urdf, 2 links, 1 joints
Links:
- link baseLink: geometry collision cylinder length=0.025 radius=0.12; collision mesh filename=plate1.obj scale=0.4 0.4 0.4
