Commit message: implement drawer_shelf_plate_stacking

File: helping_hands_rl_envs/simulators/urdf/rack2.urdf (robot description, URDF)
Before this commit: robot rack, 4 links, 3 joints
Links:
- link rack_bottom: geometry collision box size=0.05 0.1 0.01; visual box size=0.05 0.1 0.01
Joints:
- joint v2rop: origin xyz=-0.05 0 0.05 rpy=0 -1.77 0 -> xyz=-0.025 0 0.05 rpy=0 -1.57 0

File: helping_hands_rl_envs/simulators/urdf/rack_fixed.urdf (robot description, URDF)
Before this commit: robot rack, 4 links, 3 joints
Links:
- added link world
Joints:
- added joint world_to_rack: type fixed, parent world, child rack, origin xyz=0 0 0 rpy=0 0 0
