Commit message: working on bowl_spoon_cup env

File: helping_hands_rl_envs/simulators/urdf/object/cup/cup.urdf (robot description, URDF)
Before this commit: robot bowl.urdf, 1 links, 0 joints
Links:
- added link grasp, mass 0; visual box size=0.01 0.01 0.01
- link baseLink: geometry collision mesh filename=cup1.obj scale=0.1 0.1 0.1; visual mesh filename=cup1.obj scale=0.1 0.1 0.1
Joints:
- added joint base2grasp: type fixed, parent baseLink, child grasp, origin xyz=0 0 0.06 rpy=0 0 0
