Commit message: debugged covid_test_env, improving planner SR

File: helping_hands_rl_envs/simulators/urdf/object/swab/swab1.urdf (robot description, URDF)
Before this commit: robot swab, 3 links, 2 joints
Links:
- link baseLink: geometry collision mesh filename=swab_rod.obj scale=1 1 1; visual mesh filename=swab_rod.obj scale=1 1 1
- link tip: geometry collision mesh filename=swab_cotton_tip.obj scale=1 1 1; visual mesh filename=swab_cotton_tip.obj scale=1 1 1
Joints:
- joint tip2base: origin xyz=0.05 0 0 rpy=0 0 0 -> xyz=0.025 0 0 rpy=0 0 0

File: helping_hands_rl_envs/simulators/urdf/object/test_tube/test_tube1.urdf (robot description, URDF)
Before this commit: robot test_tube, 3 links, 2 joints
Links:
- link baseLink: geometry collision mesh filename=covid_test_tube_container.obj scale=1 1 1; visual mesh filename=covid_test_tube_container.obj scale=1 1 1
- link cap: geometry collision mesh filename=covid_test_tube_cap.obj scale=1 1 1; visual mesh filename=covid_test_tube_cap.obj scale=1 1 1
- link grasp: geometry visual box size=0.005 0.005 0.005
Joints:
- joint cap2base: origin xyz=0.05 0 0 rpy=0 0 0 -> xyz=0.025 0 0 rpy=0 0 0
