Commit message: improving covid_test_env planner SR

File: helping_hands_rl_envs/simulators/urdf/object/swab/swab2.urdf (robot description, URDF)
Before this commit: robot swab, 3 links, 2 joints
Links:
- link baseLink: geometry collision mesh filename=swab_rod.obj scale=2 2 2; visual mesh filename=swab_rod.obj scale=2 2 2
- link grasp: geometry visual box size=0.002 0.002 0.002
- link tip: geometry collision mesh filename=swab_cotton_tip.obj scale=2 2 2; visual mesh filename=swab_cotton_tip.obj scale=2 2 2
Joints:
- joint tip2base: origin xyz=0.075 0 0 rpy=0 0 0 -> xyz=0.05 0 0 rpy=0 0 0

File: helping_hands_rl_envs/simulators/urdf/object/test_tube/test_tube2.urdf (robot description, URDF)
Before this commit: robot test_tube, 3 links, 2 joints
Links:
- link baseLink: geometry collision mesh filename=covid_test_tube_container.obj scale=2 2 2; visual mesh filename=covid_test_tube_container.obj scale=2 2 2
- link cap: geometry collision mesh filename=covid_test_tube_cap.obj scale=2 2 2; visual mesh filename=covid_test_tube_cap.obj scale=2 2 2
- link grasp: geometry visual box size=0.01 0.01 0.01
Joints:
- joint base2cap: origin xyz=-0.075 0 0 rpy=0 0 0 -> xyz=-0.05 0 0 rpy=0 0 0
