Commit message: created test_tube, swab

File: helping_hands_rl_envs/simulators/urdf/object/swab/swab.urdf (robot description, URDF)
Before this commit: robot test_tube, 3 links, 2 joints
Links:
- removed link cap
- added link tip; collision mesh filename=swab_cotton_tip.obj scale=1 1 1; visual mesh filename=swab_cotton_tip.obj scale=1 1 1
- link baseLink: mass None -> .01; geometry collision mesh filename=swab_rod.obj scale=1 1 1; visual mesh filename=swab_rod.obj scale=1 1 1
Joints:
- removed joint cap2base
- added joint tip2base: type fixed, parent tip, child baseLink, origin xyz=0.025 0 0 rpy=0 0 0

Commit message: debugged rand perturbe rot trans covid_test env, SR 99%, scale (0.55)

File: helping_hands_rl_envs/simulators/urdf/object/swab/swab.urdf (robot description, URDF)
Before this commit: robot swab, 3 links, 2 joints
Links:
- link tip: geometry collision mesh filename=swab_tip_enlarged.obj scale=2 2 2; visual mesh filename=swab_tip_enlarged.obj scale=2 2 2
