Commit message: finished bottle_tray_env with fixed tray

File: helping_hands_rl_envs/simulators/urdf/object/bottle/bottle1.urdf (robot description, URDF)
Before this commit: robot obj, 2 links, 1 joints
Links:
- link baseLink: geometry collision cylinder length=0.16 radius=0.028; visual mesh filename=bottle1.obj scale=0.15 0.15 0.15
- link grasp: geometry 

File: helping_hands_rl_envs/simulators/urdf/object/bottle/bottle10.urdf (robot description, URDF)
Before this commit: robot obj, 2 links, 1 joints
Links:
- link baseLink: geometry collision cylinder length=0.21 radius=0.028; visual mesh filename=bottle10.obj scale=0.2 0.2 0.2
Joints:
- joint base2grasp: origin xyz=0 0 0.13 rpy=0 0 0 -> xyz=0 0 0.14 rpy=0 0 0

File: helping_hands_rl_envs/simulators/urdf/object/bottle/bottle3.urdf (robot description, URDF)
Before this commit: robot obj, 2 links, 1 joints
Links:
- link baseLink: geometry collision cylinder length=0.21 radius=0.028; visual mesh filename=bottle3.obj scale=0.23 0.23 0.2
- link grasp: geometry 
Joints:
- joint base2grasp: origin xyz=0 0 0.16 rpy=0 0 0 -> xyz=0 0 0.14 rpy=0 0 0

File: helping_hands_rl_envs/simulators/urdf/object/bottle/bottle5.urdf (robot description, URDF)
Before this commit: robot obj, 2 links, 1 joints
Links:
- link baseLink: geometry collision cylinder length=0.22 radius=0.028; visual mesh filename=bottle5.obj scale=0.2 0.2 0.2
- link grasp: geometry 
Joints:
- joint base2grasp: origin xyz=0 0 0.13 rpy=0 0 0 -> xyz=0 0 0.15 rpy=0 0 0

File: helping_hands_rl_envs/simulators/urdf/object/bottle/bottle7.urdf (robot description, URDF)
Before this commit: robot obj, 2 links, 1 joints
Links:
- link baseLink: mass 0.1 -> 0.5; geometry collision mesh filename=bottle7.obj scale=0.2 0.2 0.2; visual mesh filename=bottle7.obj scale=0.2 0.2 0.2
Joints:
- joint base2grasp: origin xyz=0 0 0.13 rpy=0 0 0 -> xyz=0 0 0.14 rpy=0 0 0

File: helping_hands_rl_envs/simulators/urdf/object/bottle/bottle8.urdf (robot description, URDF)
Before this commit: robot obj, 2 links, 1 joints
Links:
- link baseLink: geometry collision cylinder length=0.21 radius=0.028; visual mesh filename=bottle8.obj scale=0.2 0.2 0.2
Joints:
- joint base2grasp: origin xyz=0 0 0.13 rpy=0 0 0 -> xyz=0 0 0.14 rpy=0 0 0

File: helping_hands_rl_envs/simulators/urdf/object/bottle/bottle9.urdf (robot description, URDF)
Before this commit: robot obj, 2 links, 1 joints
Links:
- link baseLink: geometry collision cylinder length=0.21 radius=0.028; visual mesh filename=bottle9.obj scale=0.2 0.2 0.2
Joints:
- joint base2grasp: origin xyz=0 0 0.13 rpy=0 0 0 -> xyz=0 0 0.14 rpy=0 0 0

Commit message: shorten the bottles and increase the thickness of the box in bottle_tray

File: helping_hands_rl_envs/simulators/urdf/object/bottle/bottle1.urdf (robot description, URDF)
Before this commit: robot obj, 2 links, 1 joints
Links:
- link baseLink: mass 0.1 -> 0.5; geometry collision cylinder length=0.12 radius=0.028; visual mesh filename=bottle1.obj scale=0.15 0.15 0.12

File: helping_hands_rl_envs/simulators/urdf/object/bottle/bottle10.urdf (robot description, URDF)
Before this commit: robot obj, 2 links, 1 joints
Links:
- link baseLink: mass 0.1 -> 0.5; geometry collision cylinder length=0.168 radius=0.028; visual mesh filename=bottle10.obj scale=0.2 0.2 0.16

File: helping_hands_rl_envs/simulators/urdf/object/bottle/bottle3.urdf (robot description, URDF)
Before this commit: robot obj, 2 links, 1 joints
Links:
- link baseLink: mass 0.1 -> 0.5; geometry collision cylinder length=0.168 radius=0.028; visual mesh filename=bottle3.obj scale=0.23 0.23 0.16

File: helping_hands_rl_envs/simulators/urdf/object/bottle/bottle4.urdf (robot description, URDF)
Before this commit: robot obj, 2 links, 1 joints
Links:
- link baseLink: mass 0.1 -> 0.5; geometry collision cylinder length=0.144 radius=0.028; visual mesh filename=bottle4.obj scale=0.13 0.13 0.136

File: helping_hands_rl_envs/simulators/urdf/object/bottle/bottle5.urdf (robot description, URDF)
Before this commit: robot obj, 2 links, 1 joints
Links:
- link baseLink: mass 0.1 -> 0.5; geometry collision cylinder length=0.176 radius=0.028; visual mesh filename=bottle5.obj scale=0.2 0.2 0.16

File: helping_hands_rl_envs/simulators/urdf/object/bottle/bottle7.urdf (robot description, URDF)
Before this commit: robot obj, 2 links, 1 joints
Links:
- link baseLink: geometry collision cylinder length=0.168 radius=0.028; visual mesh filename=bottle7.obj scale=0.2 0.2 0.16

File: helping_hands_rl_envs/simulators/urdf/object/bottle/bottle8.urdf (robot description, URDF)
Before this commit: robot obj, 2 links, 1 joints
Links:
- link baseLink: mass 0.1 -> 0.5; geometry collision cylinder length=0.168 radius=0.028; visual mesh filename=bottle8.obj scale=0.2 0.2 0.16

File: helping_hands_rl_envs/simulators/urdf/object/bottle/bottle9.urdf (robot description, URDF)
Before this commit: robot obj, 2 links, 1 joints
Links:
- link baseLink: mass 0.1 -> 0.5; geometry collision cylinder length=0.168 radius=0.028; visual mesh filename=bottle9.obj scale=0.2 0.2 0.16
