Commit message: improve bumpy_box_palletizing performance; use box collision shape in pallet.urdf; implement random bump rotation

File: helping_hands_rl_envs/simulators/urdf/object/pallet/pallet.urdf (robot description, URDF)
Before this commit: robot cube.urdf, 1 links, 0 joints
Links:
- link baseLink: geometry collision box size=0.29 0.24 0.038; visual mesh filename=pallet.obj scale=0.25 0.25 0.25

Commit message: change pallet into solid for real world experiments, add _changeBoxDynamics in box_palletizing_env

File: helping_hands_rl_envs/simulators/urdf/object/pallet/pallet.urdf (robot description, URDF)
Before this commit: robot cube.urdf, 1 links, 0 joints
Links:
- link baseLink: geometry collision box size=0.29 0.24 0.03175; visual box size=0.29 0.24 0.03175

Commit message: update pallet size

File: helping_hands_rl_envs/simulators/urdf/object/pallet/pallet.urdf (robot description, URDF)
Before this commit: robot cube.urdf, 1 links, 0 joints
Links:
- link baseLink: geometry collision box size=0.3125 0.25 0.0275; visual box size=0.3125 0.25 0.0275
