Commit message: fix ur5 urdf

File: helping_hands_rl_envs/simulators/urdf/ur5/ur5_robotiq_85_gripper_fake.urdf (robot description, URDF)
Before this commit: robot assembled_robot, 25 links, 24 joints
Joints:
- joint simple_gripper_tip_joint: origin xyz=0.0 0.0 0.040 rpy=0 0 0 -> xyz=0.0 0.0 0.050 rpy=0 3.14 0
