Commit message: update default parameter, fix bug in cylinder

File: helping_hands_rl_envs/pybullet/urdf/object/cylinder.urdf (robot description, URDF)
Before this commit: robot cylinder.urdf, 1 links, 0 joints
Links:
- link baseLink: geometry collision mesh filename=cylinder.obj scale=1.2 1.2 1.2; visual mesh filename=cylinder.obj scale=1.2 1.2 1.2
