Commit message: Better panda force sensing, added collision shapes for drawer handle sides, minor other physics updates

File: bulletarm/pybullet/urdf/drawer1.urdf (robot description, URDF)
Before this commit: robot drawer, 14 links, 13 joints
Links:
- link back_wall: mass 0.05 -> 0.005
- link base_link: mass .1 -> .01
- link bottom_wall: mass 0.05 -> 0.005
- link drawer: mass .1 -> .01
- link drawer_back_wall: mass 0.05 -> 0.005
- link drawer_bottom_wall: mass 0.05 -> 0.005
- link drawer_front_wall: mass 0.05 -> 0.005
- link drawer_left_wall: mass 0.05 -> 0.005
- link drawer_obj_pos: mass 0.05 -> 0.005
- link drawer_right_wall: mass 0.05 -> 0.005
- link left_wall: mass 0.05 -> 0.005
- link right_wall: mass 0.05 -> 0.005
- link top_wall: mass 0.05 -> 0.005

File: bulletarm/pybullet/urdf/franka_panda/panda.urdf (robot description, URDF)
Before this commit: robot panda, 15 links, 14 joints
Links:
- link panda_hand: mass .81 -> .081
- link panda_left_finger: mass 0.1 -> 0.01
- link panda_leftfinger: mass 0.1 -> 0.01
- link panda_link0: mass 2.9 -> .29
- link panda_link1: mass 2.7 -> .27
- link panda_link2: mass 2.73 -> .273
- link panda_link3: mass 2.04 -> .204
- link panda_link4: mass 2.08 -> .208
- link panda_link5: mass 3 -> .3
- link panda_link6: mass 1.3 -> .13
- link panda_link7: mass .2 -> .02
- link panda_right_finger: mass 0.1 -> 0.01
- link panda_rightfinger: mass 0.1 -> 0.01
