Commit message: Initial attempt to move force-aware domains into BulletArm from old repo. Needs more rigirous testings

File: bulletarm/pybullet/urdf/franka_panda/panda.urdf (robot description, URDF)
Before this commit: robot panda, 13 links, 12 joints
Links:
- added link panda_left_finger, mass 0.1; visual box size=0.00 0.00 0.00
- added link panda_right_finger, mass 0.1; visual box size=0.0 0.0 0.0
- link panda_hand: geometry collision mesh filename=package://meshes/collision/hand.obj; visual box size=0.00 0.00 0.00
- link panda_leftfinger: geometry collision mesh filename=package://meshes/collision/finger.obj; visual box size=0.00 0.00 0.00
- link panda_rightfinger: geometry collision mesh filename=package://meshes/collision/finger.obj; visual box size=0.00 0.00 0.00
Joints:
- added joint panda_left_finger: type fixed, parent panda_hand, child panda_left_finger, origin xyz=0 0.0 0.0 rpy=0 0 0
- added joint panda_right_finger: type fixed, parent panda_hand, child panda_right_finger, origin xyz=0 0.0 0.0 rpy=0 0 0
- joint panda_finger_joint1: parent panda_hand -> panda_left_finger
- joint panda_finger_joint2: parent panda_hand -> panda_right_finger

Commit message: testing

File: bulletarm/pybullet/urdf/franka_panda/panda.urdf (robot description, URDF)
Before this commit: robot panda, 15 links, 14 joints
Links:
- link panda_hand: geometry collision mesh filename=package://meshes/collision/hand.obj; visual mesh filename=package://meshes/visual/hand.obj
- link panda_leftfinger: geometry collision mesh filename=package://meshes/collision/finger.obj; visual mesh filename=package://meshes/visual/finger.obj
- link panda_rightfinger: geometry collision mesh filename=package://meshes/collision/finger.obj; visual mesh filename=package://meshes/visual/finger.obj

Commit message: Testing longer panda fingers for drawer opening

File: bulletarm/pybullet/urdf/franka_panda/panda.urdf (robot description, URDF)
Before this commit: robot panda, 15 links, 14 joints
Links:
- link panda_leftfinger: geometry collision mesh filename=package://meshes/collision/finger.obj scale=1.0 1.0 1.5; visual mesh filename=package://meshes/visual/finger.obj scale=1.0 1.0 1.5
- link panda_rightfinger: geometry collision mesh filename=package://meshes/collision/finger.obj scale=1.0 1.0 1.5; visual mesh filename=package://meshes/visual/finger.obj scale=1.0 1.0 1.5
Joints:
- joint panda_grasptarget_hand: origin xyz=0 0 0.105 rpy=3.1415 0 1.5707 -> xyz=0 0 0.1575 rpy=3.1415 0 1.5707

Commit message: Renamed equipments to equipment. Working on pivoting domain

File: bulletarm/pybullet/urdf/franka_panda/panda.urdf (robot description, URDF)
Before this commit: robot panda, 15 links, 14 joints
Links:
- link panda_grasptarget: geometry visual box size=0.01 0.01 0.01
Joints:
- joint panda_grasptarget_hand: origin xyz=0 0 0.1575 rpy=3.1415 0 1.5707 -> xyz=0 0 0.135 rpy=3.1415 0 1.5707

Commit message: Removed visual grasp target from panda

File: bulletarm/pybullet/urdf/franka_panda/panda.urdf (robot description, URDF)
Before this commit: robot panda, 15 links, 14 joints
Links:
- link panda_grasptarget: geometry visual box size=0.0 0.0 0.0
