Commit message: More work on cabinet opening, updates to arm movement so that it can exit soon when stuck

File: bulletarm/pybullet/urdf/cabinet/cabinet.urdf (robot description, URDF)
Before this commit: robot cabinet, 6 links, 5 joints
Joints:
- joint cabinet_door_left_handle_transform: origin xyz=0.02 -0.31 0.00 rpy=0 0 0 -> xyz=-0.36 0.0 0.00 rpy=0 0 0
- joint cabinet_door_left_joint: limit lower=-1.57 upper=0 effort=1000.0 velocity=100 -> lower=0.02 upper=1.57 effort=1000.0 velocity=100
- joint cabinet_door_left_joint_fixed: origin xyz=0 0 0 rpy=0 0 0 -> xyz=0.38 -0.31 0 rpy=0 0 0
- joint cabinet_door_left_joint_fixed_2: origin xyz=0.18 -0.30 0.0 rpy=0 0 0 -> xyz=-0.20 0.0 0.0 rpy=0 0 0
