Commit message: peg insertion changes

File: bulletarm/pybullet/urdf/object/square_peg.urdf (robot description, URDF)
Before this commit: robot square_peg.urdf, 1 links, 0 joints
Links:
- link baseLink: geometry collision mesh filename=cube.obj scale=0.5 0.5 1.2; visual mesh filename=cube.obj scale=0.5 0.5 1.2
