Commit message: Made peg and holder joint fixed so peg does not rotate

File: bulletarm/pybullet/urdf/peg_insertion/round_peg/Peg.urdf (robot description, URDF)
Before this commit: robot Peg, 2 links, 1 joints
Joints:
- joint Insertion: axis 0 1 0 -> (none); type continuous -> fixed

File: bulletarm/pybullet/urdf/peg_insertion/square_peg/Peg.urdf (robot description, URDF)
Before this commit: robot Peg, 2 links, 1 joints
Joints:
- joint Insertion: axis 0 1 0 -> (none); type continuous -> fixed
